Commit message: fix(launch): finish of launch files and add config files

File: urdf/robot.urdf (robot description, URDF)
Before this commit: robot filoberta, 10 links, 9 joints
Joints:
- joint joint6: mimic (none) -> joint=gripper multiplier=-0.015 offset=-0.025
- joint joint7: mimic (none) -> joint=joint6 multiplier=1.0 offset=0.0

Commit message: feat: add xacro properies to urdf and update rviz config

File: urdf/robot.urdf (robot description, URDF)
Before this commit: robot filoberta, 10 links, 9 joints
Joints:
- joint elbow: origin xyz=0.0315 -0.101 0.0 rpy=0.0 0.0 0.0 -> xyz=${Lm} ${-L2} 0.0 rpy=0.0 0.0 0.0
- joint joint4: origin xyz=0.109 0.0 0.0 rpy=0.0 0.0 0.0 -> xyz=${L4} 0.0 0.0 rpy=0.0 0.0 0.0
- joint joint_world: origin xyz=0.0 0.0 0.0 rpy=0.0 0.0 0.0 -> (none)
- joint shoulder: origin xyz=0.0 0.0 0.0445 rpy=${-pi/2} 0.0 0.0 -> xyz=0.0 0.0 ${L1} rpy=${-pi/2} 0.0 0.0
- joint waist: origin xyz=0.0 0.0 0.0445 rpy=0.0 0.0 0.0 -> xyz=0.0 0.0 ${0.08945-L1} rpy=0.0 0.0 0.0
- joint wrist: origin xyz=0.101 0.0 0.0 rpy=0.0 0.0 0.0 -> xyz=${L3} 0.0 0.0 rpy=0.0 0.0 0.0

Commit message: refactor: change package name
-change name rviz launch to visualize.launch
-add missing video

File: urdf/robot.urdf (robot description, URDF)
Before this commit: robot filoberta, 10 links, 9 joints
Links:
- link finger_1: geometry visual mesh filename=package://px100_description/meshes/px100_8_gripper_finger.s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 scale=0.001 0.001 0.001
- link finger_2: geometry visual mesh filename=package://px100_description/meshes/px100_8_gripper_finger.s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 scale=0.001 0.001 0.001
- link gripper_bar: geometry visual mesh filename=package://px100_description/meshes/px100_7_gripper_bar.stl scale=0.001 0.001 0.001
- link link0: geometry visual mesh filename=package://px100_description/meshes/px100_1_base.stl scale=0.001 0.001 0.001
- link link1: geometry visual mesh filename=package://px100_description/meshes/px100_2_shoulder.stl scale=0.001 0.001 0.001
- link link2: geometry visual mesh filename=package://px100_description/meshes/px100_3_upper_arm.stl scale=0.001 0.001 0.001
- link link3: geometry visual mesh filename=package://px100_description/meshes/px100_4_forearm.stl scale=0.001 0.001 0.001
- link link4: geometry visual mesh filename=package://px100_description/meshes/px100_5_gripper.stl scale=0.001 0.001 0.001
- link prop: geometry visual mesh filename=package://px100_description/meshes/px100_6_gripper_prop.stl scale=0.001 0.001 0.001

Commit message: fix: urdf link 1

File: urdf/robot.urdf (robot description, URDF)
Before this commit: robot filoberta, 10 links, 9 joints
Joints:
- joint joint6: origin xyz=${0.08605-0.109} 0.0 0.0 rpy=${pi/2} ${pi} 0.0 -> xyz=${0.08605-L4} 0.0 0.0 rpy=${pi/2} ${pi} 0.0
- joint joint7: origin xyz=${0.08605-0.109} 0.0 0.0 rpy=${-pi/2} ${pi} 0.0 -> xyz=${0.08605-L4} 0.0 0.0 rpy=${-pi/2} ${pi} 0.0

Commit message: fix: change in urdf frames
- change urdf frames to match with dh convention
- add joint state publisher gui to visualize launch file

File: urdf/robot.urdf (robot description, URDF)
Before this commit: robot filoberta, 10 links, 9 joints
Joints:
- joint elbow: origin xyz=${Lm} ${-L2} 0.0 rpy=0.0 0.0 0.0 -> xyz=${Lm} ${-L2} 0.0 rpy=0.0 0.0 ${-atan2(L2,Lm)}
- joint joint4: origin xyz=${L4} 0.0 0.0 rpy=0.0 0.0 0.0 -> xyz=${L4} 0.0 0.0 rpy=${-pi/2} 0.0 ${-pi/2}
- joint joint6: mimic joint=gripper multiplier=-0.015 offset=-0.025 -> joint=gripper multiplier=-0.008 offset=-0.0265; origin xyz=${0.08605-L4} 0.0 0.0 rpy=${pi/2} ${pi} 0.0 -> xyz=0.0 0.0 ${0.08605-L4} rpy=0.0 ${pi/2} 0.0
- joint joint7: origin xyz=${0.08605-L4} 0.0 0.0 rpy=${-pi/2} ${pi} 0.0 -> xyz=0.0 0.0 ${0.08605-L4} rpy=0.0 ${pi/2} ${pi}
- joint wrist: origin xyz=${L3} 0.0 0.0 rpy=0.0 0.0 0.0 -> xyz=${L3*cos(atan2(L2,Lm))} ${L3*sin(atan2(L2,Lm))} 0.0 rpy=0.0 0.0 ${atan2(L2,Lm)}
